File: KiCAD/FreeEEG128-alpha.kicad_pcb (KiCad board)
At the start: 4 copper layers, 70 x 70 mm, 165 parts, among them J1 Conn_02x02_Odd_Even, J100 Conn_01x02, J101 Conn_01x02, J103 USB_B_Micro, J104 Conn_01x02, J105 Conn_01x02, J2 Conn_02x02_Odd_Even, J201 Conn_02x20_Odd_Even, J202 Conn_02x20_Odd_Even, J203 Conn_02x20_Odd_Even, J204 Conn_02x20_Odd_Even, J205 Conn_02x20_Odd_Even, J206 Conn_02x20_Odd_Even, J207 Conn_02x20_Odd_Even, J208 Conn_02x20_Odd_Even, J81 Conn_02x03_Odd_Even, J84 Conn_02x03_Odd_Even, J99 USB_B_Micro, SW1 SW_Push, SW2 SW_Push, T1 750315371, U1 LSM6DS3, U101 ADS131M08IRSN, U102 ADS131M08IRSN, U103 ADS131M08IRSN, U104 ADS131M08IRSN, U105 ADS131M08IRSN, U106 ADS131M08IRSN, U107 ADS131M08IRSN, U108 ADS131M08IRSN, U109 ADS131M08IRSN, U110 ADS131M08IRSN, U111 ADS131M08IRSN, U112 ADS131M08IRSN, U113 ADS131M08IRSN, U114 ADS131M08IRSN, U115 ADS131M08IRSN, U116 ADS131M08IRSN, U15 ISO7341c, U16 ADUM1402BRWZ, U17 ADuM3160, U18 STM32H743ZITx, U19 SN6505B, U2 REF2025, U21 473521001, U22 LP5907, U6 LP5907, U7 FXO-SM7_OSC-SMD7050_short, U8 LP5907, Y1 32768Hz, Y2 16MHz

Commit message: Add files via upload
Parts:
- added J301: Conn_02x04_Odd_Even, Connector_PinSocket_1.27mm:PinSocket_2x04_P1.27mm_Vertical, F.Cu at (16.1, 1.90)
- added J302: Conn_02x04_Odd_Even, Connector_PinHeader_1.27mm:PinHeader_2x04_P1.27mm_Vertical, F.Cu at (-1.90, 17.4)
- added J303: Conn_02x04_Odd_Even, Connector_PinSocket_1.27mm:PinSocket_2x04_P1.27mm_Vertical, F.Cu at (-16.1, -1.90)
Connections:
- net ADC15_19_SCLK renamed ADC13_19_SCLK
- net ADC15_20_DOUT renamed ADC13_20_DOUT
- net ADC15_21_DIN renamed ADC13_21_DIN
- net ADC8_20_DOUT renamed ADC5_20_DOUT
- net ISO_USB_8_GND1 renamed ISO_USB_2_GND1
Routing:
- net MCU_23_RCC_OSC_IN: track 8.40 -> 41.7 mm, vias 1 -> 3
- net MCU_10_PF0_I2C2_SDA: track 0.00 -> 24.5 mm, vias 0 -> 2
- net MCU_11_PF1_I2C2_SCL: track 0.00 -> 22.8 mm, vias 0 -> 2
- net CRYSTAL_3_OUT: track 3.55 -> 24.2 mm, vias 0 -> 2
- net AINREF+: track 307.5 -> 327.6 mm, vias 4 -> 5
- net MCU_118_PD4_ADC1_SYNC/RESET: track 3.28 -> 22.0 mm, vias 1 -> 2
- net CRYSTAL_4_Vin: track 3.50 -> 19.0 mm, vias 0 -> 2
- net AINREF-: track 353.4 -> 365.6 mm
- net ACC_12_CS: track 304.6 -> 316.0 mm, vias 17 -> 18
- net ADC5_19_SCLK: track 67.7 -> 74.2 mm
- net ADC5_20_DOUT: track 42.4 -> 47.8 mm
- net AVDD_1_IN: track 129.4 -> 134.4 mm, vias 5 -> 6
- net ADC10_15_AVDD: track 394.7 -> 399.6 mm
- net ADC10_26_DVDD: track 218.2 -> 222.0 mm, vias 17 -> 16
- net ADC5_21_DIN: track 37.7 -> 40.8 mm
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