File: KiCAD/FreeEEG128-alpha.kicad_sch (KiCad schematic)
At the start: 34 parts, among them J1 Conn_02x02_Odd_Even, J14 Conn_01x02, J15 Conn_01x02, J16 Conn_01x02, J17 Conn_01x02, J18 Conn_01x02, J19 Conn_01x02, J2 Conn_02x02_Odd_Even, J20 Conn_01x02, J201 Conn_02x20_Odd_Even, J202 Conn_02x20_Odd_Even, J203 Conn_02x20_Odd_Even, J204 Conn_02x20_Odd_Even, J205 Conn_02x20_Odd_Even, J206 Conn_02x20_Odd_Even, J207 Conn_02x20_Odd_Even, J208 Conn_02x20_Odd_Even, J21 Conn_01x02, J22 Conn_01x02, J23 Conn_01x02, J24 Conn_01x02, J25 Conn_01x02, J26 Conn_01x02, J27 Conn_01x02, J28 Conn_01x02, SW1 SW_Push, SW2 SW_Push

Commit message: Add files via upload
Parts:
- added J301, J303: Conn_02x04_Odd_Even, Connector_PinSocket_1.27mm:PinSocket_2x04_P1.27mm_Vertical, symbol Connector_Generic:Conn_02x04_Odd_Even
- added J302: Conn_02x04_Odd_Even, Connector_PinHeader_1.27mm:PinHeader_2x04_P1.27mm_Vertical, symbol Connector_Generic:Conn_02x04_Odd_Even
Connections:
- net ACC_12_CS: now also J301.5 (Pin_5), J302.2 (Pin_2)
- net ACC_6_GND: now also J301.1 (Pin_1), J303.2 (Pin_2)
- net ADC10_15_AVDD: now also J303.4 (Pin_4)
- net ADC10_16_SYNC/RESET: now also J301.6 (Pin_6), J302.3 (Pin_3)
- net ADC10_26_DVDD: now also J303.6 (Pin_6)
- net AINREF+: now also J301.2 (Pin_2)
- net AINREF-: now also J301.4 (Pin_4)
- net AVDD_1_IN: now also J301.3 (Pin_3)
- net CRYSTAL_3_OUT: now also J302.6 (Pin_6)
- net CRYSTAL_4_Vin: now also J302.1 (Pin_1)
- net MCU_10_PF0_I2C2_SDA: now also J303.5 (Pin_5)
- net MCU_118_PD4_ADC1_SYNC/RESET: now also J302.4 (Pin_4)
- net MCU_11_PF1_I2C2_SCL: now also J303.3 (Pin_3)
- net MCU_23_RCC_OSC_IN: now also J302.5 (Pin_5), J303.1 (Pin_1)
